Commit message: made compatible with CHAMP

File: cheetah_description/xacro/mini_cheetah.urdf (robot description, URDF)
Before this commit: robot mini_cheetah, 20 links, 19 joints
Links:
- removed link base
- removed link roty
- removed link rotz
Joints:
- removed joint rot_x
- removed joint rot_y
- removed joint rot_z
- joint FL_calf_joint: axis 0 0 1 -> 0 1 0; origin xyz=0.209 0.0 0 rpy=0.0 0 0.0 -> xyz=0 0 -0.209 rpy=0.0 0 0.0
- joint FL_foot_fixed: origin xyz=0.18 0 0 -> xyz=0 0 -0.18
- joint FL_hip_joint: axis 0 0 1 -> 1 0 0; origin xyz=0.19 0.049 0.0 rpy=1.5708 0 1.5708 -> xyz=0.19 0.049 0.0 rpy=0 0 0
- joint FL_thigh_joint: axis 0 0 1 -> 0 1 0; origin xyz=0.062 0 0.00 rpy=0.0 1.5708 0.0 -> xyz=0 0.062 0 rpy=0.0 0 0.0
- joint FR_calf_joint: axis 0 0 1 -> 0 1 0; origin xyz=0.209 0 0  rpy=0.0 0 0.0 -> xyz=0 0 -0.209  rpy=0.0 0 0.0
- joint FR_foot_fixed: origin xyz=0.18 0 0 -> xyz=0 0 -0.18
- joint FR_hip_joint: axis 0 0 1 -> 1 0 0; origin xyz=0.19 -0.049 0.0 rpy=1.57079632679 0 1.57079632679 -> xyz=0.19 -0.049 0.0 rpy=0 0 0
- joint FR_thigh_joint: axis 0 0 1 -> 0 1 0; origin xyz=-0.062 0 0.00 rpy=0.0 1.5708 0.0 -> xyz=0 -0.062 0 rpy=0.0 0.0 0.0
- joint RL_calf_joint: axis 0 0 1 -> 0 1 0; origin xyz=0.209 0.0 0 rpy=0.0 0 0.0 -> xyz=0 0 -0.209  rpy=0.0 0 0.0
- joint RL_foot_fixed: origin xyz=0.18 0 0 -> xyz=0 0 -0.18
- joint RL_hip_joint: axis 0 0 1 -> 1 0 0; origin xyz=-0.19 0.049 0.0 rpy=1.5708 0 1.5708 -> xyz=-0.19 0.049 0.0 rpy=0 0 0
- joint RL_thigh_joint: axis 0 0 1 -> 0 1 0; origin xyz=0.062 0 0.00 rpy=0.0 1.5708 0.0 -> xyz=0 0.062 0 rpy=0.0 0.0 0.0
- joint RR_calf_joint: axis 0 0 1 -> 0 1 0; origin xyz=0.209 0.0 0 rpy=0.0 0 0.0 -> xyz=0 0 -0.209  rpy=0.0 0 0.0
- joint RR_foot_fixed: origin xyz=0.18 0 0 -> xyz=0 0 -0.18
- joint RR_hip_joint: axis 0 0 1 -> 1 0 0; origin xyz=-0.19 -0.049 0.0 rpy=1.57079632679 0 1.57079632679 -> xyz=-0.19 -0.049 0.0 rpy=0 0 0
- joint RR_thigh_joint: axis 0 0 1 -> 0 1 0; origin xyz=-0.062 0 0.00 rpy=0.0 1.5708 0.0 -> xyz=0 -0.062 0 rpy=0.0 0 0.0
